Commit message: Update: added the laser range finder to the robot model

File: urdf/graph_slam_bot.xacro (robot description, xacro)
@@ -144,4 +144,35 @@
 		</visual>
 	</link>
-	<joint name=""
+	<joint name="camera_joint">
+		<origin xyz="0.2 0 0" rpy="0 0 0"/>
+		<child link="camera"/>
+		<parent link="chassis"/>
+	</joint>
+	<!-- Laser Rangefinder-->
+	<link name="hokuyo">
+		<inertial>
+			<mass value="0.1"/>
+			<origin xyz="0 0 0" rpy="0 0 0"/>
+			<inertia
+				ixx="1e-6" ixy="0" ixz="0"
+				iyy="1e-6" iyz="0"
+				izz="1e-6"
+			/>
+		</inertial>
+		<collision>
+			<origin xyz="0 0 0" rpy="0 0 0"/>
+			<geometry>
+				<box size="0.1 0.1 0.1"/>
+			</geometry>
+		</collision>
+		<visual>
+			<origin xyz="0 0 0" rpy="0 0 0"/>
+			<mesh filename="package://graph_slam_bot/meshes/hokuyo.dae"/>
+		</visual>
+	</link>
+	<joint name="hokuyo_joint">
+		<origin xyz="0.15 0 0.1" rpy="0 0 0"/>
+		<child link="hokuyo"/>
+		<parent link="chassis"/>
+	</joint>
 </robot>

Commit message: Updated: changed camera and lrf joints from continuous to fixed

File: urdf/graph_slam_bot.xacro (robot description, xacro)
@@ -1,4 +1,5 @@
 <?xml version="1.0"?>
 <robot name="graph_slam_bot" xmlns:xacro="http://www.ros.org/wiki/xacro">
+	<xacro:include filename="$(find graph_slam_bot)/urdf/graph_slam_bot.gazebo"/>
 	<link name="robot_footprint"></link>
 	<joint name="robot_footprint_joint" type="fixed">
@@ -144,5 +145,5 @@
 		</visual>
 	</link>
-	<joint name="camera_joint">
+	<joint type="continuous" name="camera_joint">
 		<origin xyz="0.2 0 0" rpy="0 0 0"/>
 		<child link="camera"/>
@@ -168,8 +169,10 @@
 		<visual>
 			<origin xyz="0 0 0" rpy="0 0 0"/>
-			<mesh filename="package://graph_slam_bot/meshes/hokuyo.dae"/>
+			<geometry>
+				<mesh filename="package://graph_slam_bot/meshes/hokuyo.dae"/>
+			</geometry>
 		</visual>
 	</link>
-	<joint name="hokuyo_joint">
+	<joint type="continuous" name="hokuyo_joint">
 		<origin xyz="0.15 0 0.1" rpy="0 0 0"/>
 		<child link="hokuyo"/>

Commit message: Add: updated the launch file to launch RVIZ

File: urdf/graph_slam_bot.xacro (robot description, xacro)
@@ -145,5 +145,5 @@
 		</visual>
 	</link>
-	<joint type="continuous" name="camera_joint">
+	<joint type="fixed" name="camera_joint">
 		<origin xyz="0.2 0 0" rpy="0 0 0"/>
 		<child link="camera"/>
@@ -174,5 +174,5 @@
 		</visual>
 	</link>
-	<joint type="continuous" name="hokuyo_joint">
+	<joint type="fixed" name="hokuyo_joint">
 		<origin xyz="0.15 0 0.1" rpy="0 0 0"/>
 		<child link="hokuyo"/>

Commit message: Update: robot is not compiling properly - need to diagnose the problem agaist a working model

File: urdf/graph_slam_bot.xacro (robot description, xacro)
@@ -13,5 +13,5 @@
 		<inertial>
 			<mass value="15.0"/>
-			<origin xyz="0 0 0" rpy="0 0 0"/>
+			<origin xyz="0.0 0 0" rpy="0 0 0"/>
 			<inertia
 				ixx="0.1" ixy="0.0" ixz="0.0"
@@ -20,5 +20,5 @@
 			/>
 		</inertial>
-		<collision name='chassis_collision'>
+		<collision name='collision'>
 			<origin xyz="0 0 0" rpy="0 0 0"/>
 			<geometry>

Commit message: Update: launch files configured with RGBD camera and removed RVIZ launch from world launch

File: urdf/graph_slam_bot.xacro (robot description, xacro)
@@ -20,5 +20,5 @@
 			/>
 		</inertial>
-		<collision name='collision'>
+		<collision name='chassis_collision'>
 			<origin xyz="0 0 0" rpy="0 0 0"/>
 			<geometry>
@@ -68,5 +68,5 @@
 			/>
 		</inertial>
-		<collision name="left_wheel_collision">
+		<collision>
 			<origin xyz="0 0 0" rpy="0 1.5707 1.5707"/>
 			<geometry>
@@ -74,5 +74,5 @@
 			</geometry>
 		</collision>
-		<visual name="left_wheel_visual">
+		<visual>
 			<origin xyz="0 0 0" rpy="0 1.5707 1.5707"/>
 			<geometry>
@@ -83,6 +83,6 @@
 	<joint type="continuous" name="left_wheel_hinge">
 		<origin xyz="0 0.15 0" rpy="0 0 0"/>
+		<parent link="chassis"/>
 		<child link="left_wheel"/>
-		<parent link="chassis"/>
 		<axis xyz="0 1 0" rpy="0 0 0"/>
 		<limit effort="10000" velocity="1000"/>
@@ -100,5 +100,5 @@
 			/>
 		</inertial>
-		<collision name="right_wheel_collision">
+		<collision>
 			<origin xyz="0 0 0" rpy="0 1.5707 1.5707"/>
 			<geometry>
@@ -106,5 +106,5 @@
 			</geometry>
 		</collision>
-		<visual name="left_wheel_visual">
+		<visual>
 			<origin xyz="0 0 0" rpy="0 1.5707 1.5707"/>
 			<geometry>
@@ -115,6 +115,6 @@
 	<joint type="continuous" name="right_wheel_hinge">
 		<origin xyz="0 -0.15 0" rpy="0 0 0"/>
+		<parent link="chassis"/>
 		<child link="right_wheel"/>
-		<parent link="chassis"/>
 		<axis xyz="0 1 0" rpy="0 0 0"/>
 		<limit effort="10000" velocity="1000"/>
@@ -147,6 +147,6 @@
 	<joint type="fixed" name="camera_joint">
 		<origin xyz="0.2 0 0" rpy="0 0 0"/>
+		<parent link="chassis"/>
 		<child link="camera"/>
-		<parent link="chassis"/>
 	</joint>
 	<!-- Laser Rangefinder-->
@@ -176,6 +176,6 @@
 	<joint type="fixed" name="hokuyo_joint">
 		<origin xyz="0.15 0 0.1" rpy="0 0 0"/>
+		<parent link="chassis"/>
 		<child link="hokuyo"/>
-		<parent link="chassis"/>
 	</joint>
 </robot>

Commit message: Update: minor modifications to the RVIZ config and robot model files

File: urdf/graph_slam_bot.xacro (robot description, xacro)
@@ -2,4 +2,5 @@
 <robot name="graph_slam_bot" xmlns:xacro="http://www.ros.org/wiki/xacro">
 	<xacro:include filename="$(find graph_slam_bot)/urdf/graph_slam_bot.gazebo"/>
+	<!-- Robot Base -->
 	<link name="robot_footprint"></link>
 	<joint name="robot_footprint_joint" type="fixed">
@@ -8,5 +9,5 @@
 		<child link="chassis"/>
 	</joint>
-	<!-- Robot Chassis-->
+	<!-- Robot Chassis -->
 	<link name="chassis">
 		<pose>0 0 0.1 0 0 0</pose>
@@ -150,4 +151,18 @@
 		<child link="camera"/>
 	</joint>
+	<!-- generate an optical frame
+      http://www.ros.org/reps/rep-0103.html#suffix-frames
+      so that ros and opencv can operate on the camera frame correctly
+      -->
+    <link name="camera_link_optical">
+  	</link>
+  	<joint name="camera_optical_joint" type="fixed">
+    <!-- these values have to be these values otherwise the gazebo camera
+        image won't be aligned properly with the frame it is supposedly
+        originating from -->
+    	<origin xyz="0 0 0" rpy="${-pi/2} 0 ${-pi/2}"/>
+    	<parent link="camera"/>
+    	<child link="camera_link_optical"/>
+  	</joint>
 	<!-- Laser Rangefinder-->
 	<link name="hokuyo">

Commit message: Update: change to material colour on robot chassis for RVIZ

File: urdf/graph_slam_bot.xacro (robot description, xacro)
@@ -1,5 +1,8 @@
 <?xml version="1.0"?>
 <robot name="graph_slam_bot" xmlns:xacro="http://www.ros.org/wiki/xacro">
+	<!-- Import the Gazebo plugin file (i.e. udacity_bot.gazebo) -->
 	<xacro:include filename="$(find graph_slam_bot)/urdf/graph_slam_bot.gazebo"/>
+	<!-- Import Rviz colors -->
+  	<xacro:include filename="$(find graph_slam_bot)/urdf/materials.xacro"/>
 	<!-- Robot Base -->
 	<link name="robot_footprint"></link>
@@ -32,4 +35,5 @@
 				<box size="0.4 0.2 0.1"/>
 			</geometry>
+			<material name="blue"/>
 		</visual>
 		<collision name='back_caster_collision'>
@@ -80,4 +84,5 @@
 				<cylinder radius="0.1" length="0.05"/>
 			</geometry>
+			<material name="green"/>
 		</visual>
 	</link>
@@ -112,4 +117,5 @@
 				<cylinder radius="0.1" length="0.05"/>
 			</geometry>
+			<material name="green"/>
 		</visual>
 	</link>
@@ -144,4 +150,5 @@
 				<box size="0.05 0.05 0.05"/>
 			</geometry>
+			<material name="red"/>
 		</visual>
 	</link>
